Commit message: Testing Odom correction for ICP procesing on the fly

File: charle_description/urdf/charle.xacro (robot description, xacro)
@@ -120,5 +120,10 @@
 			</geometry>
  	 </collision>
-      <xacro:default_inertial mass="0.5"/>
+                  <inertial>
+                       <mass value="0.01" />
+                       <inertia ixx="1" ixy="0.0" ixz="0.0"
+                                iyy="1" iyz="0.0"
+                                izz="0.001" />
+               </inertial>
   </link>
   <joint name="sonarDato_to_sonar" type="fixed">

Commit message: Merge with previous project and update

File: charle_description/urdf/charle.xacro (robot description, xacro)
@@ -146,5 +146,5 @@
     <parent link="sonar"/>
     <child link="laserDato"/>
-    <origin rpy="1.57 3.14 3.14" xyz="-0.0 -0.075 -0.02"/>
+    <origin rpy="1.57 0 0" xyz="-0.0 -0.075 -0.02"/>
   </joint>
   <link name="laserDato">
