Commit message: Checking hough and improving some node parameters

File: charle_description/urdf/charle.urdf (robot description, URDF)
Before this commit: robot charle_xacro, 9 links, 8 joints
Links:
- removed link head
- added link head_link; visual mesh filename=package://charle_description/urdf/AVORA_head_stl.STL scale=0.001 0.001 0.001
- link base_footprint: mass 0.0001 -> None
- link base_link: mass 0.5 -> 0.1
- link sonar: mass 0.5 -> 0.01
- link sonarDato: mass None -> 0.1; geometry collision cylinder length=0.02 radius=0.02; visual cylinder length=0.02 radius=0.02
- link thruster_1: mass 0.5 -> 0.1
- link thruster_2: mass 0.5 -> 0.1
Joints:
- joint head_to_servo_head: child head -> head_link
- joint laserDato_to_sonar: origin xyz=-0.0 -0.075 -0.02 rpy=1.57 3.14 3.14 -> xyz=-0.0 -0.075 -0.02 rpy=1.57 0 0
- joint sonarDato_to_sonar: origin xyz=-0.0 -0.075 -0.02 rpy=1.57 0 0 -> xyz=-0.0 -0.075 -0.02 rpy=0 0 0

File: charle_description/urdf/charle.xacro (robot description, xacro)
@@ -5,5 +5,5 @@
     	xmlns:interface="http://playerstage.sourceforge.net/gazebo/xmlschema/#interface"
 	name="charle_xacro">
-	<xacro:include filename="$(find charle_description)/urdf/charle.gazebo" />
+    <xacro:include filename="$(find charle_description)/urdf/charle.gazebo" />
 	<xacro:property name="length_thruster" value="0.2" />
 	<xacro:property name="radius_thruster" value="0.01" />
@@ -13,5 +13,5 @@
                        <inertia ixx="1" ixy="0.0" ixz="0.0"
                                 iyy="1" iyz="0.0"
-                                izz="0.01" />
+                                izz="1" />
                </inertial>
 	</xacro:macro>
@@ -28,5 +28,4 @@
 				</geometry>
 			</collision>
-		<xacro:default_inertial mass="0.0001"/>
  	</link>
 	<gazebo reference="base_footprint">
@@ -54,5 +53,5 @@
 			</geometry>
 	 </collision>
-	 <xacro:default_inertial mass="0.5"/>
+	 <xacro:default_inertial mass="0.1"/>
   </link>
  	<joint name="base_to_thruster_1" type="continuous">
@@ -75,5 +74,5 @@
 			</geometry>
 		</collision>
-		<xacro:default_inertial mass="0.5"/>
+		<xacro:default_inertial mass="0.1"/>
  	</link>
  <joint name="base_to_thruster_2" type="continuous">
@@ -83,19 +82,19 @@
    <axis xyz="0 0 1" />
  </joint>
- 	<link name="thruster_2">
-   		<visual>
-     			<geometry>
-       				<cylinder length="${length_thruster}" radius="${radius_thruster}"/>
-     			</geometry>
-			<!-- <origin rpy="0 1.5 0" xyz="0.1 0.1 0"/> -->
-			<origin rpy="0 0 0" xyz="0 0 0"/>
-		</visual>
-		<collision>
-			<geometry>
-       				<cylinder length="${length_thruster}" radius="${radius_thruster}"/>
-			</geometry>
-		</collision>
-		<xacro:default_inertial mass="0.5"/>
- 	</link>
+  <link name="thruster_2">
+      <visual>
+          <geometry>
+              <cylinder length="${length_thruster}" radius="${radius_thruster}"/>
+          </geometry>
+      <!-- <origin rpy="0 1.5 0" xyz="0.1 0.1 0"/> -->
+      <origin rpy="0 0 0" xyz="0 0 0"/>
+    </visual>
+    <collision>
+      <geometry>
+              <cylinder length="${length_thruster}" radius="${radius_thruster}"/>
+      </geometry>
+    </collision>
+    <xacro:default_inertial mass="0.1"/>
+  </link>
   <joint name="sonar_to_base_link" type="revolute">
     <parent link="base_link"/>
@@ -103,5 +102,5 @@
     <origin rpy="1.5707 0 0" xyz="-0.0 -0 -0.205"/>
     <axis xyz="1 0 0" />
-    <limit effort ="1000.0" lower="-1.57" upper="1.57" velocity="0.5"/>
+    <limit effort ="10000.0" lower="-1.57" upper="1.57" velocity="0.5"/>
   </joint>
   <link name="sonar">
@@ -120,27 +119,55 @@
 			</geometry>
  	 </collision>
-                  <inertial>
-                       <mass value="0.01" />
-                       <inertia ixx="1" ixy="0.0" ixz="0.0"
-                                iyy="1" iyz="0.0"
-                                izz="0.001" />
+               <inertial>
+                       <mass value="1" />
+                       <inertia ixx="0" ixy="0.0" ixz="0.0"
+                                iyy="0" iyz="0.0"
+                                izz="0" />
                </inertial>
   </link>
-  <joint name="sonarDato_to_sonar" type="fixed">
+  <joint name="sonarDato_to_sonar" type="continuous">
     <parent link="sonar"/>
     <child link="sonarDato"/>
     <origin rpy="1.57 0 0" xyz="-0.0 -0.075 -0.02"/>
-  </joint>
-  <link name="sonarDato">
-    <visual>
-	<origin rpy="0 0 0" xyz="-0.0 -0.0 0.0"/>
-      <geometry>
-        <cylinder length="0.02" radius="0.02"/>
-      </geometry>
-      <material name="blue">
-     	<color rgba="0 0 .8 1"/>
-      </material>
-    </visual>
-  </link>
+    <axis xyz="0 0 1" />
+    <limit effort ="1000.0" velocity="1000000"/>
+  </joint>
+ <link name="sonarDato">
+    <visual>
+	   <origin rpy="0 0 0" xyz="-0.0 -0.0 0.0"/>
+      <geometry>
+        <cylinder length="0.01" radius="0.01"/>
+      </geometry>
+      <material name="blue">
+     	<color rgba="0 0 .8 1"/>
+      </material>
+    </visual>
+             <collision>
+      <geometry>
+              <cylinder length="0.01" radius="0.01"/>
+      </geometry>
+   </collision>
+       <xacro:default_inertial mass="0.00001"/>
+  </link>
+  <transmission name="tran1">
+    <type>transmission_interface/SimpleTransmission</type>
+    <joint name="sonar_to_base_link">
+      <hardwareInterface>EffortJointInterface</hardwareInterface>
+    </joint>
+    <actuator name="sonar_servo">
+       <hardwareInterface>EffortJointInterface</hardwareInterface>
+      <mechanicalReduction>1</mechanicalReduction>
+    </actuator>
+  </transmission>
+  <!--<transmission name="tran2">
+    <type>transmission_interface/SimpleTransmission</type>
+    <joint name="sonarDato_to_sonar">
+      <hardwareInterface>PositionJointInterface</hardwareInterface>
+    </joint>
+    <actuator name="sonarDato_servo">
+       <hardwareInterface>PositionJointInterface</hardwareInterface>
+      <mechanicalReduction>1</mechanicalReduction>
+    </actuator>
+  </transmission>-->
   <joint name="laserDato_to_sonar" type="fixed">
     <parent link="sonar"/>
@@ -150,10 +177,10 @@
   <link name="laserDato">
     <visual>
-	<origin rpy="0 0 0" xyz="-0.0 -0.0 0.0"/>
+  <origin rpy="0 0 0" xyz="-0.0 -0.0 0.0"/>
       <geometry>
         <cylinder length="0.02" radius="0.02"/>
       </geometry>
       <material name="blue">
-     	<color rgba="0 0 .8 1"/>
+      <color rgba="0 0 .8 1"/>
       </material>
     </visual>
@@ -179,12 +206,12 @@
   <joint name="head_to_servo_head" type="revolute">
     <parent link="servo_head"/>
-    <child link="head"/>
+    <child link="head_link"/>
     <origin rpy="0 0 3.14" xyz="0 0 0.04"/>
     <axis xyz="0 0 1" />
     <limit effort ="1000.0" lower="0.8" upper="2.4" velocity="0.5"/>
   </joint>
-  <link name="head">
-    <visual>
-	<origin rpy="1.54 0 -1.54" xyz="0 0 0" />
+  <link name="head_link">
+    <visual>
+	    <origin rpy="1.54 0 -1.54" xyz="0 0 0" />
       <geometry>
         <mesh filename="package://charle_description/urdf/AVORA_head_stl.STL" scale="0.001 0.001 0.001"/>
